File: Hardware/pcb.brd (EAGLE design)
At the start: 46 x 35 mm, 105 parts, among them IC1 BQ25180YBGR, IC2 DRV2605YZFR, IC3 BMA423, IC9 RT6160AWSC, J1 503480-2400, J2 TC2030-IDC, J4 KH-TYPE-C-16P, Q1 20V/4.2A/52mΩ/1.4W, Q3 SI1308EDL-T1-GE3, U1 NRF52840_QF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

Commit message: Add files via upload
Parts:
- C23, C27, C29, C30, C31, C32, C34, C37, C38, C42: device InkTime_v5:GRM011R60J152KE01L_1_0201 -> InkTime_v5:ERA-1AEB3401C_0201
- L1, L2, L3: device InkTime_v5:NORDIC_NRF_2_RESC0402_L -> InkTime_v5:NORDIC_NRF_2_RESC0402_N
- moved R5 3.78 mm to (66.3, 109.7)
- moved C30 3.02 mm to (67.8, 109.7), turned to 180 degrees
- moved SJ1 2.85 mm to (89.1, 110.2), turned to 211.8 degrees
- moved R_TYPE_SEL 2.25 mm to (85.5, 109.1), turned to 126.9 degrees
- moved TP_VBAT 1.73 mm to (91.5, 114.3), turned to 180 degrees
- moved J4 1.52 mm to (71.1, 140.4)
- moved C2-EP-DR 1.50 mm to (66.1, 119.0)
- moved C22 1.04 mm to (80.6, 123.5)
- moved TP_BAT_GND 1.00 mm to (92.1, 119.8)
- moved TP_SWO 0.92 mm to (76.9, 119.3)
- moved R1_USB 0.85 mm to (73.0, 133.0)
- moved TP_GND 0.85 mm to (59.5, 114.2)
- moved R2_USB 0.82 mm to (69.7, 133.2)
- moved C4 0.81 mm to (80.4, 125.1)
- moved TP_OP 0.71 mm to (54.1, 115.1)
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Routing:
- net GND: track 29.7 -> 15.8 mm, vias 4 -> 3
- net VBUS/1.5D: track 20.6 -> 16.6 mm, vias 0 -> 2
- net P0.13/1.5D: track 1.35 -> 4.05 mm
- net N$16: track 24.3 -> 21.7 mm, vias 4 -> 2
- net 3V3/1.7D: track 52.9 -> 51.2 mm
- net N$10: track 21.8 -> 23.4 mm
- net VBAT/1.2A: track 6.28 -> 7.68 mm
- net N$9: track 5.13 -> 6.15 mm
- net N$22: track 3.11 -> 4.05 mm
- net RESET: track 21.2 -> 21.9 mm
- net DP: track 9.17 -> 8.55 mm
- net DN: track 10.4 -> 11.0 mm
- net DEC3: track 1.81 -> 1.28 mm
- net N$7: track 3.63 -> 4.14 mm
Other:
- board text added: "3V3"
- board text added: "GND"
- board text added: "ON"
- board text added: "OP"
- board text added: "RESET"
- board text added: "SCL"
- board text added: "SDA"
- board text added: "SWDCLK"
- board text added: "SWDIO"
- board text added: "SWO"
- board text added: "VBAT"
- board text added: "VREG"
